File: kicad/AND_OR.sch (KiCad schematic (older format))
At the start: 44 parts, among them J601 power, Q601 BC547, Q602 BC547

Commit message: tests and doc ok
still need some scoring options
Parts:
- added R612: 100k, Resistor_THT:R_Axial_DIN0204_L3.6mm_D1.6mm_P7.62mm_Horizontal, symbol Device:R
Connections:
- net GND: now also R612.2
- net at D621.1 (K), D622.1 (K), D623.1 (K)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: now also R612.1
Other:
- note added: "LTSPICE - OK"
