File: kicad/Score_Counter.sch (KiCad schematic (older format))
At the start: 16 parts, among them J501 Reset, J701 power, Q501 BC547, Q502 BC547, Q503 BC547, U501 LM393, U502 4017

Commit message: tests and doc ok
still need some scoring options
Parts:
- added D701, D702: 1N4148, Diode_THT:D_DO-35_SOD27_P7.62mm_Horizontal, symbol Diode:1N4148
- added Q504: BC547, Package_TO_SOT_THT:TO-92_Inline_Wide, symbol Transistor_BJT:BC547
- added R508, R509, R510: 10k, Resistor_THT:R_Axial_DIN0204_L3.6mm_D1.6mm_P7.62mm_Horizontal, symbol Device:R
- R507: value 1k -> 10k
Connections:
- net +5V: now also R508.1, R510.1; no longer R507.1
- net Edge: now also R509.2; no longer Q503.1 (C), R508.2, U502.14 (CLK)
- net GND: now also D701.2 (A), D702.2 (A), Q504.3 (E)
- net Pad+: now also U501.3 (+); no longer U501.2 (-)
- net Pad-: now also U501.6 (_); no longer U501.5 (+)
- net Pos_Y: now also U501.2 (-), U501.5 (+); no longer U501.3 (+), U501.6 (_)
- net at R507.2, U501.1, U501.7: no longer Q503.2 (B)
- net sheet5C868ABE/A1 renamed AND_OR/A1
- net sheet5C868ABE/B1 renamed AND_OR/B1
- net sheet5C868ABE/C1 renamed AND_OR/C1
- net sheet5C868ABE/D1 renamed AND_OR/D1
- net sheet5C868ABE/E1 renamed AND_OR/E1
- net sheet5C868ABE/F1 renamed AND_OR/F1
- net sheet5C868ABE/G1 renamed AND_OR/G1
- net sheet5C868ABE/H1 renamed AND_OR/H1
- net sheet5C868ABE/I1 renamed AND_OR/I1
- net sheet5C868ABE/J1 renamed AND_OR/J1
- new net: D701.1 (K), Q503.2 (B), R507.1, R508.2
- new net: D702.1 (K), Q504.2 (B), R509.1, R510.2
- new net Goal: Q503.1 (C), Q504.1 (C), R508.2, U502.14 (CLK)
Other:
- note added: "AND ball on the edge"
- note added: "Ball outside the pad area"
- note added: "If the current score\nis the one displayed"
- note added: "LTSPICE - OK"
- note added: "THEN add a point"
- note added: "VISUAL - OK"
- moved on the sheet: J501, J502, JP501, Q501, Q502, Q503, R501, R502, R503, R504, R505, R506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

Commit message: Small fixes and more documentation
Other:
- note added: "REALITY - OK"
- note removed: "VISUAL - OK"
