File: kicad/full/osc.sch (KiCad schematic (older format))
At the start: 36 parts, among them J201 power, Q201 BC547, Q202 2N3819, Q203 BC547, U201 TL082, U202 TL082, U203 TL082

Commit message: Changed some parts to sourcable ones
Parts:
- Q202: value 2N3819 -> J111; symbol Device:Q_NJFET_DGS -> Device:Q_NJFET_GSD
- R213: value 100 -> 330
Connections:
- net +15V: now also Q202.3 (D); no longer Q202.1 (D)
- net at C203.2, R212.2, R213.2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: now also Q202.1 (G); no longer Q202.2 (G)
- net at R213.1: now also Q202.2 (S); no longer Q202.3 (S)
Other:
- note added: "7-8mA"
- note removed: "7mA"
Changed lines of the file:
@@
 AR Path="/5C71D21F/5C8FB93C" Ref="R213"  Part="1"
 F 0 "R213" H 2720 3696 50  0000 L CNN
-F 1 "100" H 2720 3605 50  0000 L CNN
+F 1 "330" H 2720 3605 50  0000 L CNN
 F 2 "Resistor_THT:R_Axial_DIN0204_L3.6mm_D1.6mm_P7.62mm_Horizontal" V 2580 3650 50  0001 C CNN
 F 3 "~" H 2650 3650 50  0001 C CNN
@@
 	2650 3450 2650 3500
 $Comp
-L Device:Q_NJFET_DGS Q?
+L Device:Q_NJFET_GSD Q?
 U 1 1 5C8FB934
 P 2550 3250
@@
 AR Path="/5C71D21F/5C8FB934" Ref="Q202"  Part="1"
 F 0 "Q202" H 2741 3296 50  0000 L CNN
-F 1 "2N3819" H 2741 3205 50  0000 L CNN
+F 1 "J111" H 2741 3205 50  0000 L CNN
 F 2 "Package_TO_SOT_THT:TO-92_Inline_Wide" H 2750 3350 50  0001 C CNN
 F 3 "~" H 2550 3250 50  0001 C CNN
@@
 	0    -1   -1   0
 $EndComp
-Text Notes 2650 4050 1    50   ~ 0
-7mA
+Text Notes 2750 4050 1    50   ~ 0
+7-8mA
 Text Notes 3950 3500 0    50   ~ 0
 18kHz

Commit message: Tested goal_detector, small fix
Parts:
- gave numbers to parts that had none: 1
Changed lines of the file:
@@
 AR Path="/5C78AC26/5EAD3FA1" Ref="R?"  Part="1"
 AR Path="/5C7A25BC/5EAD3FA1" Ref="R?"  Part="1"
-AR Path="/5C71D21F/5EAD3FA1" Ref="R?"  Part="1"
-F 0 "R?" H 1920 4596 50  0000 L CNN
+AR Path="/5C71D21F/5EAD3FA1" Ref="R218"  Part="1"
+F 0 "R218" H 1920 4596 50  0000 L CNN
 F 1 "100k" H 1920 4505 50  0000 L CNN
 F 2 "Resistor_THT:R_Axial_DIN0204_L3.6mm_D1.6mm_P7.62mm_Horizontal" V 1780 4550 50  0001 C CNN
@@
 $EndComp
 $Comp
-L power:-15V #PWR?
+L power:-15V #PWR0192
 U 1 1 5EAD48A8
 P 1850 4750
-AR Path="/5C71D21F/5EAD48A8" Ref="#PWR?"  Part="1"
+AR Path="/5C71D21F/5EAD48A8" Ref="#PWR0192"  Part="1"
 AR Path="/5C722BDF/5EAD48A8" Ref="#PWR?"  Part="1"
-F 0 "#PWR?" H 1850 4850 50  0001 C CNN
+F 0 "#PWR0192" H 1850 4850 50  0001 C CNN
 F 1 "-15V" H 1865 4923 50  0000 C CNN
 F 2 "" H 1850 4750 50  0001 C CNN
@@
 $EndComp
 $Comp
-L power:GND #PWR?
+L power:GND #PWR0193
 U 1 1 5EB0338B
 P 5700 5250
-AR Path="/5C71D21F/5EB0338B" Ref="#PWR?"  Part="1"
+AR Path="/5C71D21F/5EB0338B" Ref="#PWR0193"  Part="1"
 AR Path="/5C722BDF/5EB0338B" Ref="#PWR?"  Part="1"
-F 0 "#PWR?" H 5700 5000 50  0001 C CNN
+F 0 "#PWR0193" H 5700 5000 50  0001 C CNN
 F 1 "GND" H 5705 5077 50  0000 C CNN
 F 2 "" H 5700 5250 50  0001 C CNN
@@
 P 5700 4000
 AR Path="/5EB07399" Ref="#PWR?"  Part="1"
-AR Path="/5C71D21F/5EB07399" Ref="#PWR?"  Part="1"
-F 0 "#PWR?" H 5700 3850 50  0001 C CNN
+AR Path="/5C71D21F/5EB07399" Ref="#PWR0194"  Part="1"
+F 0 "#PWR0194" H 5700 3850 50  0001 C CNN
 F 1 "+5V" H 5715 4173 50  0000 C CNN
 F 2 "" H 5700 4000 50  0001 C CNN
@@
 	5700 4950 5700 5250
 $Comp
-L power:GND #PWR?
+L power:GND #PWR0195
 U 1 1 5EB24896
 P 5350 5250
-AR Path="/5C71D21F/5EB24896" Ref="#PWR?"  Part="1"
+AR Path="/5C71D21F/5EB24896" Ref="#PWR0195"  Part="1"
 AR Path="/5C722BDF/5EB24896" Ref="#PWR?"  Part="1"
-F 0 "#PWR?" H 5350 5000 50  0001 C CNN
+F 0 "#PWR0195" H 5350 5000 50  0001 C CNN
 F 1 "GND" H 5355 5077 50  0000 C CNN
 F 2 "" H 5350 5250 50  0001 C CNN

Commit message: Tested oscillator
Parts:
- Q202: symbol Device:Q_NJFET_GSD -> Device:Q_NJFET_DSG
Connections:
- net +15V: now also Q202.1 (D); no longer Q202.3 (D)
- net at C203.2, R212.2, R213.2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: now also Q202.3 (G); no longer Q202.1 (G)
Changed lines of the file:
@@
 	2650 3450 2650 3500
 $Comp
-L Device:Q_NJFET_GSD Q?
+L Device:Q_NJFET_DSG Q?
 U 1 1 5C8FB934
 P 2550 3250

Commit message: new ramp design
Parts:
- removed R218: 100k, Resistor_THT:R_Axial_DIN0204_L3.6mm_D1.6mm_P7.62mm_Horizontal, symbol Device:R
- added D205: 1N4148, Diode_THT:D_DO-35_SOD27_P7.62mm_Horizontal, symbol Diode:1N4148
- added Q203: BC547, Package_TO_SOT_THT:TO-92_Inline_Wide, symbol Transistor_BJT:BC547
- added R216: 10k, Resistor_THT:R_Axial_DIN0204_L3.6mm_D1.6mm_P7.62mm_Horizontal, symbol Device:R
- added unit 1 of U202
- C203: value 10n -> 1n
- R212: value 100 -> 270
- R213: value 330 -> 3k3
- R214: value 7k5 -> 6k8
- renumbered D205 to D206, Q203 to Q204, R216 to R217, R217 to R218, U202 to U201
Connections:
- net +5V: now also R216.1
- net -15V: now also D205.1 (K); no longer C203.1, Q201.3 (E)
- net GND: now also U201.5 (+); no longer U201.3 (+)
- net Sin: now also U202.1, U202.2 (-); no longer R208.2, R209.1, RV201.1, RV201.2, U201.1
- net reset: now also Q201.2 (B), R211.2, Q203.2 (B); no longer R211.1, R215.2, R217.1, U203.7
- net at R206.2, R207.2: now also U201.6 (-); no longer U201.2 (-)
- net at D203.2 (A): now also C203.1, Q201.3 (E), Q203.3 (E); no longer R211.2
- net at D204.1 (K): now also D205.2 (A); no longer Q201.2 (B)
- new net: R208.2, R209.1, RV201.1, RV201.2, U201.7, U202.3 (+)
- new net: R211.1, R215.2, U203.7
- new net: Q203.1 (C), R216.2, R217.1
Other:
- note added: "1mA"
- note added: "35kHz"
- note added: "Dephaser"
- note added: "Gain"
- note added: "I used 7k5 and 5k"
- note added: "OPA dropout compensation"
- note added: "REALITY - Good enough"
- note added: "REALITY - OK"
- note added: "Wien oscillator"
- note removed: "18kHz"
- note removed: "7-8mA"
- note removed: "LTSPICE - OK"
- moved on the sheet: C201, C202, C204, D201, D202, D203, D204, D206, Q204, R201, R202, R203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

Commit message: Small correction
Parts:
- R218: value 10k -> 2k7
- renumbered D205 to D201, D204 to D202, D201 to D204, D202 to D205, R203 to R202, R202 to R203, R212 to R206, R213 to R207, R206 to R208, R207 to R209, R214 to R210, R215 to R211, R208 to R212, R209 to R213, R211 to R214, R210 to R215
Connections:
- net -15V: now also C203.1
- net at D203.2 (A), Q201.3 (E), Q203.3 (E): no longer C203.1
Other:
- note added: "+ they are not rail to rail"
- note added: "Really slow rise time\nwith 10k"
- note added: "Touching the slew-rate limit"
- moved on the sheet: D201, D202, D203
