File: kicad/full/AND_OR.sch (KiCad schematic (older format))
At the start: 45 parts, among them J601 power, Q601 BC547, Q602 BC547

Commit message: Refactor
Parts:
- renumbered R612 to R611, R611 to R612
