File: kicad/full/Ball.sch (KiCad schematic (older format))
At the start: 33 parts, among them J901 power, K301 G5V-1, Q301 BC547, Q302 BC547, Q303 BC557, Q304 2N3819, Q305 BC547, U301 TL082, U302 TL082, U303 TL082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

Commit message: Changed some parts to sourcable ones
Parts:
- removed U304, U305: DG470, Package_DIP:DIP-8_W7.62mm, symbol Analog_Switch:DG419LDJ
- added U304: DG470, Package_SO:MSOP-8_3x3mm_P0.65mm, symbol telec:DG470
- added U305: DG468, Package_SO:TSOP-6_1.65x3.05mm_P0.95mm, symbol telec:DG468
- Q304: value 2N3819 -> J111; symbol Device:Q_NJFET_DGS -> Device:Q_NJFET_GSD
- R305: value 100k -> 330k
Connections:
- net +15V: now also U304.4 (V+), U305.5 (V+)
- net -15V: now also U304.7 (V-), U305.2 (V-)
- net Ball_pos: now also U305.1
- net GND: now also U304.3 (GND), U304.5 (~EN), U305.4 (GND)
- net Score: now also U305.3
- net at C302.2, Q302.1 (C), R305.2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: now also Q304.1 (G); no longer Q304.2 (G)
- net at C303.1, R310.1, U302.6 (-): now also U305.6
- net at Q303.1 (C): now also Q304.3 (D); no longer Q304.1 (D)
- net at R305.1: now also Q304.2 (S); no longer Q304.3 (S)
- no-connect marks 1 -> 0
Other:
- note added: "16uA"
- note added: "~~+2V/pulse"

Commit message: Tested goal_detector, small fix
Connections:
- net at K301.1, R307.1, U301.7: now also U304.8
- net at K301.10, R306.1, U301.1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: now also U304.2
- net at K301.5, K301.6, R310.2: now also U304.1
- net at K301.9, Q305.1 (C), R308.1: now also U304.6

Commit message: Refactor
Parts:
- removed R313, R314, R315: 10k, Resistor_THT:R_Axial_DIN0204_L3.6mm_D1.6mm_P7.62mm_Horizontal, symbol Device:R
- removed U303: TL082, Package_SO:SOIC-8_3.9x4.9mm_P1.27mm, symbol Amplifier_Operational:TL082
- renumbered U304 to U303, U305 to U304
Other:
- note removed: "Sum position and shape"
- note removed: "X or Y value"
- moved on the sheet: C901, C902, C903, D901, D902, J901, K901, Q901, Q902, Q903, Q904, Q905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
