File: kicad/full/Score_Counter.sch (KiCad schematic (older format))
At the start: 22 parts, among them J501 Reset, J701 power, Q501 BC547, Q502 BC547, Q503 BC547, Q504 BC547, U501 LM393, U502 4017

Commit message: Tested goal_detector, small fix
Parts:
- added C501: 1u, Capacitor_THT:CP_Radial_D5.0mm_P2.50mm, symbol Device:CP
Connections:
- net GND: now also C501.2
- net Goal: now also C501.1
Other:
- note added: "Small filter"
- note removed: "LTSPICE - OK"
- moved on the sheet: J502, JP501, R511, U502

Commit message: Refactor
Parts:
- renumbered D702 to D701, D701 to D702, J501 to J502, Q504 to Q503, Q503 to Q504, R509 to R507, R507 to R508, R510 to R509, R508 to R510, R508 to R511
