File: kicad/full/pong.sch (KiCad schematic (older format))
At the start: 37 parts, among them J101 power, J102 Y_F, J103 X_F, J104 X, J105 Y, J106 Z, U101 L7805, U102 L7905, U103 TL082, U104 TL082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

Commit message: Tested goal_detector, small fix
Other:
- note added: "REALITY - OK"
Changed lines of the file:
@@
 Wire Notes Line
 	10550 5200 10550 5300
+Text Notes 8000 6250 0    50   ~ 0
+REALITY - OK
 $EndSCHEMATC

Commit message: Refactor
Parts:
- removed J102: Y_F, Connector_PinSocket_2.54mm:PinSocket_1x01_P2.54mm_Vertical, symbol Connector:Conn_01x01_Female
- removed J103: X_F, Connector_PinSocket_2.54mm:PinSocket_1x01_P2.54mm_Vertical, symbol Connector:Conn_01x01_Female
- removed R101, R102, R103, R104, R105, R106, R107, R108: R, Resistor_THT:R_Axial_DIN0204_L3.6mm_D1.6mm_P7.62mm_Horizontal, symbol Device:R
- removed R109, R112: 1k, Resistor_THT:R_Axial_DIN0204_L3.6mm_D1.6mm_P7.62mm_Horizontal, symbol Device:R
- removed R110, R111: 100, Resistor_THT:R_Axial_DIN0204_L3.6mm_D1.6mm_P7.62mm_Horizontal, symbol Device:R
- removed R113, R114, R115, R116, R117, R118, R119, R120: 100k, Resistor_THT:R_Axial_DIN0204_L3.6mm_D1.6mm_P7.62mm_Horizontal, symbol Device:R
- removed RV101, RV102: R_POT, Connector_PinHeader_2.54mm:PinHeader_1x03_P2.54mm_Vertical, symbol Device:R_POT
- removed U103, U104, U109: TL082, Package_SO:SOIC-8_3.9x4.9mm_P1.27mm, symbol Amplifier_Operational:TL082
- removed U105, U106, U107: DG445, Package_DIP:DIP-16_W7.62mm, symbol Analog_Switch:DG412xJ
- removed U108: 4017, Package_DIP:DIP-16_W7.62mm_LongPads, symbol 4xxx:4017
- renumbered J106 to J102, J105 to J103
Connections:
- no-connect marks 4 -> 0
Other:
- note removed: "Output multiplexer"
- note removed: "Select sequently which\noutput to display"
- note removed: "Shape the ramp for \nthe lines of the scores"
- note removed: "Shape the ramp for the pads"
- note removed: "Sum position and shape of the pads"
- note removed: "User input 1 (aka PAD1)"
- note removed: "User input 2 (aka PAD2)"
- moved on the sheet: J101, J102, J103, J104, U101, U102
